File: pcb/addon-ac-dimmer.sch (KiCad schematic (older format))
At the start: 41 parts, among them J1 Screw_Terminal_01x05, J2 Conn_01x02_Male ZMCT, J3 Conn_01x05_Male, J4 Conn_01x05_Male RIGHT, J5 Programm header, Q1 BT136-600D, Q2 BT136-600D, Q5 2N3904, U1 HLK-PM05, U2 MOC3052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

Commit message: Repository cleanup
Parts:
- removed C3, C5: 4.7uF, Capacitor_SMD:C_0805_2012Metric_Pad1.15x1.40mm_HandSolder, symbol Device:C
- removed C4, C6: 1uF, Capacitor_SMD:C_0805_2012Metric_Pad1.15x1.40mm_HandSolder, symbol Device:C
- removed U1: HLK-PM05, Power_Supply:HLK-PM03, symbol sensor_board-rescue:HLK-PM03-Power_Supplies
- removed U5: AMS1117-3.3, Package_TO_SOT_SMD:SOT-223-3_TabPin2, symbol Regulator_Linear:AMS1117-3.3
- added PS?: HLK-PM03, Converter_ACDC:Converter_ACDC_HiLink_HLK-PMxx, symbol Converter_ACDC:HLK-PM03
- added R16, R17: 180 0.25W 200v, Resistor_SMD:R_1210_3225Metric_Pad1.42x2.65mm_HandSolder, symbol Device:R
- C1: Vendor (none) -> C152975
- C2: Vendor (none) -> C191532
- C7: Vendor (none) -> C128353
- C8: value 100nF -> 100nF 450v; Vendor (none) -> C106025
- D1: Vendor (none) -> C184882
- D2: Vendor (none) -> C83867
- F1: value Glass fuse 10mm 3A -> Glass fuse 10mm 4A; Vendor (none) -> C140492
- J1: Vendor (none) -> C163149,C163148
- Q1, Q2: Vendor (none) -> C130426
- Q5, U4: Vendor (none) -> C115444
- R1, R2: value 360 -> 180 0.25W 200v; Vendor (none) -> C171148
- R10: footprint Resistor_SMD:R_0805_2012Metric_Pad1.15x1.40mm_HandSolder -> Resistor_SMD:R_1206_3216Metric_Pad1.30x1.75mm_HandSolder; Vendor (none) -> C175514
- R11, R13, R8: Vendor (none) -> C95781
- R12: value 50 -> 100
- R14: Vendor (none) -> C103904
- R15: value R -> DNS; Vendor (none) -> C103904
- R6, R7: value 220K -> 220K 0.25W 200v; Vendor (none) -> C352118
- U2, U3: Vendor (none) -> C115471
- U6: value ATTINY1614-SSFR -> ATTINY414-SSNR; Vendor (none) -> C189365
- U7: Vendor (none) -> C184383
Connections:
- net +3V3: now also PS?.4 (+Vout); no longer J4.1 (Pin_1)
- net +5V: no longer J4.2 (Pin_2)
- net GND: now also PS?.3 (-Vout); no longer J4.3 (Pin_3)
- net LINE: now also PS?.1 (AC/L)
- net NEUT: now also J1.2 (Pin_2), PS?.2 (AC/N); no longer J1.4 (Pin_4)
- net SW_1_LINE: now also J1.3 (Pin_3); no longer J1.5 (Pin_5)
- net at Q1.1 (A1): now also J1.5 (Pin_5); no longer J1.2 (Pin_2)
- net at R1.1: now also R16.1; no longer U2.6
- net at R3.1: now also U6.4 (AIN6/PA6); no longer U6.5 (AIN7/PA7)
- net at Q2.1 (A1): now also J1.4 (Pin_4); no longer J1.3 (Pin_3)
- net at R2.1: now also R17.1; no longer U3.6
- net at R4.1: now also U6.5 (AIN7/PA7); no longer U6.4 (AIN6/PA6)
- net at C1.1, R6.1: now also D2.1 (~~); no longer D2.2 (~~)
- net at R5.2, U4.5: now also U6.2 (AIN4/PA4); no longer U6.3 (AIN5/PA5)
- net at C1.2, R7.1: now also D2.2 (~~); no longer D2.1 (~~)
- net at J2.1 (Pin_1), R12.2: now also U6.3 (AIN5/PA5); no longer U6.2 (AIN4/PA4)
- net at C8.2: now also U7.1; no longer U7.2
- net at R10.2: now also U7.2; no longer U7.1
- new net: R16.2, U2.6
- new net: R17.2, U3.6
- no-connect marks 4 -> 7
Other:
- moved on the sheet: C8, R1, R10, R2, R6, R7
